Commit message: update gazebo model and create node controller
now it's possible to launch a controller node, this node allows to
control some part of the robot easily.

File: ros/pouco2000_gazebo/urdf/test.urdf.xacro (robot description, xacro)
@@ -5,4 +5,5 @@
     <xacro:property name="depth" value="0.2" />
     <xacro:property name="n_lvl" value="2" />
+    <xacro:property name="free_space" value="0.001" />
     <xacro:property name="level_depth" value="0.1" />
     <xacro:property name="headlight_front_width" value="0.05" />
@@ -10,9 +11,16 @@
     <xacro:property name="headlight_front_depth" value="0.2" />
     <xacro:property name="headlight_front_angle" value="${pi/8}" />
+    <xacro:property name="headlight_front_base_width" value="0.10"/>
     <xacro:property name="headlight_bottom_width" value="0.05" />
     <xacro:property name="headlight_bottom_height" value="0.5" />
     <xacro:property name="headlight_bottom_depth" value="0.05" />
     <xacro:property name="wheel_len" value="0.1"/>
-    <xacro:property name="wheel_rad" value="0.15" />
+    <xacro:property name="wheel_rad" value="0.15"/>
+    <xacro:property name="wheel_len" value="0.1"/>
+    <xacro:property name="wheel_rad" value="0.15"/>
+    <xacro:property name="fork_n" value="5"/>
+    <xacro:property name="fork_len" value="0.25"/>
+    <xacro:property name="fork_rad" value="0.02"/>
+    <xacro:property name="fork_base_width" value="0.10"/>
     <!-- colors definitions -->
     <material name="blue">
@@ -79,7 +87,7 @@
         </link>
          <joint name="headlight_front_${prefix}_joint" type="fixed">
-            <parent link="level_0_link"/>
+            <parent link="headlight_front_base_link"/>
             <child link="headlight_front_${prefix}_link"/>
-            <origin xyz="${(width + headlight_front_width)/2} ${reflect * headlight_front_height} 0.0"/>
+            <origin xyz="${(headlight_front_base_width + headlight_front_width )/2} ${reflect * headlight_front_height} 0.0"/>
         </joint>
         <gazebo reference="headlight_front_${prefix}_link">
@@ -91,5 +99,5 @@
             <visual>
                 <geometry>
-                        <box size="${headlight_bottom_width} ${headlight_bottom_height} ${headlight_bottom_depth}" />
+                    <box size="${headlight_bottom_width} ${headlight_bottom_height} ${headlight_bottom_depth}" />
                 </geometry>
                 <material name="red"/>
@@ -103,10 +111,45 @@
             <xacro:default_inertial mass="0.05"/>
         </link>
-         <joint name="headlight_back_${lvl}_joint" type="fixed">
+        <joint name="headlight_back_${lvl}_joint" type="prismatic">
+            <axis rpy="0 0 0" xyz="1 0 0"/>
             <parent link="level_${lvl}_link"/>
             <child link="headlight_back_${lvl}_link"/>
-            <origin xyz="${-1*(width + headlight_bottom_width)/2} 0.0 0.0"/>
+            <limit effort="10" lower="${-1 * headlight_bottom_width}" upper="0" velocity="0.5"/>
+            <origin xyz="${-1*(width - headlight_bottom_width)/2 + free_space} 0.0 0.0"/>
         </joint>
         <gazebo reference="headlight_back_${lvl}_link">
+            <material>Gazebo/Red</material>
+        </gazebo>
+        <transmission name="headlight_back_${lvl}_trans">
+            <type>transmission_interface/SimpleTransmission</type>
+            <actuator name="headlight_back_${lvl}_motor">
+                <mechanicalReduction>1</mechanicalReduction>
+            </actuator>
+            <joint name="headlight_back_${lvl}_joint">
+                <hardwareInterface>PositionJointInterface</hardwareInterface>
+            </joint>
+        </transmission>
+    </xacro:macro>
+    <xacro:macro name="fork" params="lvl">
+        <link name="fork_${lvl}_link">
+            <visual>
+                <geometry>
+                        <cylinder length="${fork_len}" radius="${fork_rad}"/>
+                </geometry>
+                <material name="red"/>
+            </visual>
+            <collision>
+                <geometry>
+                    <cylinder length="${fork_len}" radius="${fork_rad}"/>
+                </geometry>
+            </collision>
+            <xacro:default_inertial mass="0.05"/>
+        </link>
+         <joint name="fork_${lvl}_joint" type="fixed">
+            <parent link="fork_base_link"/>
+            <child link="fork_${lvl}_link"/>
+            <origin rpy="0 ${pi/2} 0" xyz="${(fork_len+fork_base_width)/2} ${(height * (lvl+1-1/2)/fork_n) -height/2} 0.0"/>
+        </joint>
+        <gazebo reference="fork_${lvl}_link">
             <material>Gazebo/Red</material>
         </gazebo>
@@ -160,7 +203,7 @@
         </visual>
         <collision>
-        <geometry>
-                <box size="${width} ${height} ${depth}" />
-        </geometry>
+            <geometry>
+                    <box size="${width} ${height} ${depth}" />
+            </geometry>
         </collision>
         <xacro:default_inertial mass="10"/>
@@ -172,5 +215,38 @@
     <xacro:level lvl="1" color="gray"/>
     <xacro:headlight_front prefix="left" reflect="1"/>
-    <xacro:headlight_front prefix="right" reflect="-1"/>*
+    <xacro:headlight_front prefix="right" reflect="-1"/>
+    <link name="headlight_front_base_link">
+        <visual>
+        <geometry>
+                <box size="${headlight_front_base_width} ${height} ${depth/10}"/>
+        </geometry>
+        <material name="blue"/>
+        </visual>
+        <collision>
+                <geometry>
+                    <box size="${headlight_front_base_width} ${height} ${depth/10}"/>
+                </geometry>
+        </collision>
+        <xacro:default_inertial mass="1"/>
+    </link>
+    <joint name="headlight_front_base_joint" type="prismatic">
+        <axis rpy="0 0 0" xyz="1 0 0"/>
+        <parent link="level_0_link"/>
+        <child link="headlight_front_base_link"/>
+        <limit effort="10" lower="0" upper="${headlight_front_width}" velocity="0.5"/>
+        <origin xyz="${(width - headlight_front_base_width)/2 - headlight_front_width - free_space} 0.0 0.0"/>
+    </joint>
+    <transmission name="headlight_front_base_trans">
+        <type>transmission_interface/SimpleTransmission</type>
+        <actuator name="headlight_front_base_motor">
+            <mechanicalReduction>1</mechanicalReduction>
+        </actuator>
+        <joint name="headlight_front_base_joint">
+            <hardwareInterface>PositionJointInterface</hardwareInterface>
+        </joint>
+    </transmission>
+    <gazebo reference="beacon_base_link">
+            <material>Gazebo/Black</material>
+    </gazebo>
     <xacro:headlight_back lvl="0"/>
     <xacro:headlight_back lvl="1"/>
@@ -179,4 +255,48 @@
     <xacro:wheel side="left" updown="bottom" reflect_side="1" reflect_updown="-1"/>
     <xacro:wheel side="right" updown="bottom" reflect_side="-1" reflect_updown="-1"/>
+    <link name="fork_base_link">
+        <visual>
+            <geometry>
+                <box size="${fork_base_width} ${height} ${depth/10}"/>
+            </geometry>
+        <material name="blue"/>
+        </visual>
+        <collision>
+            <geometry>
+                  <box size="${fork_base_width} ${height} ${depth/10}"/>
+            </geometry>
+        </collision>
+        <xacro:default_inertial mass="1"/>
+    </link>
+    <transmission name="fork_base_trans">
+        <type>transmission_interface/SimpleTransmission</type>
+        <actuator name="fork_base_motor">
+            <mechanicalReduction>1</mechanicalReduction>
+        </actuator>
+        <joint name="fork_base_joint">
+        <hardwareInterface>PositionJointInterface</hardwareInterface>
+        </joint>
+    </transmission>
+    <joint name="fork_base_joint" type="prismatic">
+        <axis rpy="0 0 0" xyz="1 0 0"/>
+        <parent link="base_link"/>
+        <child link="fork_base_link"/>
+        <limit effort="10" lower="0" upper="${fork_len}" velocity="0.5"/>
+        <origin xyz="${(width - fork_base_width)/2 - fork_len - free_space} 0 0.0"/>
+    </joint>
+    <transmission name="base_beacon_trans_trans">
+        <type>transmission_interface/SimpleTransmission</type>
+        <actuator name="$base_beacon_trans_motor">
+            <mechanicalReduction>1</mechanicalReduction>
+        </actuator>
+        <joint name="base_beacon_trans_joint">
+        <hardwareInterface>PositionJointInterface</hardwareInterface>
+        </joint>
+    </transmission>
+    <xacro:fork lvl="0"/>
+    <xacro:fork lvl="1"/>
+    <xacro:fork lvl="2"/>
+    <xacro:fork lvl="3"/>
+    <xacro:fork lvl="4"/>
     <link name="beacon_base_link">
         <visual>
@@ -271,4 +391,4 @@
         <robotNamespace>/</robotNamespace>
         </plugin>
-  </gazebo>
+    </gazebo>
 </robot>
