Commit message: clean gazebo package and comment
rename files of pouco2000_gazebo package and add some comments

File: ros/pouco2000_gazebo/urdf/pouco2000.urdf.xacro (robot description, xacro)
@@ -1,3 +1,4 @@
 <robot name="simple_robot" xmlns:xacro="http://ros.org/wiki/xacro">
+    <!-- definition properties -->
     <xacro:property name="pi" value="3.1415" />
     <xacro:property name="width" value="1" />
@@ -42,4 +43,6 @@
     <color rgba="1 1 0 1"/>
     </material>
+    <!-- macros definition -->
+    <!-- macro: default_inertial -->
     <xacro:macro name="default_inertial" params="mass">
         <inertial>
@@ -49,4 +52,5 @@
         </inertial>
     </xacro:macro>
+    <!-- macro: level -->
     <xacro:macro name="level" params="lvl color">
         <link name="level_${lvl}_link">
@@ -70,4 +74,5 @@
         </joint>
     </xacro:macro>
+    <!-- macro: headlight_front -->
     <xacro:macro name="headlight_front" params="prefix reflect">
         <link name="headlight_front_${prefix}_link">
@@ -95,4 +100,5 @@
         </gazebo>
     </xacro:macro>
+    <!-- macro: headlight_back -->
     <xacro:macro name="headlight_back" params="lvl">
         <link name="headlight_back_${lvl}_link">
@@ -131,4 +137,5 @@
         </transmission>
     </xacro:macro>
+    <!-- macro: fork -->
     <xacro:macro name="fork" params="lvl">
         <link name="fork_${lvl}_link">
@@ -155,4 +162,5 @@
         </gazebo>
     </xacro:macro>
+    <!-- macro: wheel -->
     <xacro:macro name="wheel" params="side updown reflect_side reflect_updown">
         <link name="wheel_${side}_${updown}_link">
@@ -195,4 +203,6 @@
         </transmission>
     </xacro:macro>
+    <!-- definition links -->
+    <!-- link: base_link -->
     <link name="base_link">
         <visual>
@@ -212,6 +222,8 @@
         <material>Gazebo/DarkGrey</material>
     </gazebo>
+    <!-- links: level -->
     <xacro:level lvl="0" color="gray"/>
     <xacro:level lvl="1" color="gray"/>
+    <!-- links: headlight_front -->
     <xacro:headlight_front prefix="left" reflect="1"/>
     <xacro:headlight_front prefix="right" reflect="-1"/>
@@ -246,13 +258,17 @@
         </joint>
     </transmission>
+    <!-- links: headlight_back -->
+    <xacro:headlight_back lvl="0"/>
+    <xacro:headlight_back lvl="1"/>
+    <!-- links: beacon -->
     <gazebo reference="beacon_base_link">
             <material>Gazebo/Black</material>
     </gazebo>
-    <xacro:headlight_back lvl="0"/>
-    <xacro:headlight_back lvl="1"/>
+    <!-- links: wheel -->
     <xacro:wheel side="left" updown="top" reflect_side="1" reflect_updown="1"/>
     <xacro:wheel side="right" updown="top" reflect_side="-1" reflect_updown="1"/>
     <xacro:wheel side="left" updown="bottom" reflect_side="1" reflect_updown="-1"/>
     <xacro:wheel side="right" updown="bottom" reflect_side="-1" reflect_updown="-1"/>
+    <!-- links: fork -->
     <link name="fork_base_link">
         <visual>
@@ -285,13 +301,4 @@
         <origin xyz="${(width - fork_base_width)/2 - fork_len - free_space} 0 0.0"/>
     </joint>
-    <transmission name="base_beacon_trans_trans">
-        <type>transmission_interface/SimpleTransmission</type>
-        <actuator name="$base_beacon_trans_motor">
-            <mechanicalReduction>1</mechanicalReduction>
-        </actuator>
-        <joint name="base_beacon_trans_joint">
-        <hardwareInterface>PositionJointInterface</hardwareInterface>
-        </joint>
-    </transmission>
     <xacro:fork lvl="0"/>
     <xacro:fork lvl="1"/>
@@ -299,4 +306,5 @@
     <xacro:fork lvl="3"/>
     <xacro:fork lvl="4"/>
+    <!-- links: beacon -->
     <link name="beacon_base_link">
         <visual>

Commit message: add antenna in the front of the robot

File: ros/pouco2000_gazebo/urdf/pouco2000.urdf.xacro (robot description, xacro)
@@ -24,4 +24,7 @@
     <xacro:property name="fork_rad" value="0.02"/>
     <xacro:property name="fork_base_width" value="0.10"/>
+    <xacro:property name="antenna_len" value="0.2"/>
+    <xacro:property name="antenna_rad" value="0.01"/>
+    <xacro:property name="antenna_space" value="0.1"/>
     <!-- colors definitions -->
     <material name="blue">
@@ -395,4 +398,30 @@
         <origin rpy="0 0 0" xyz="0.2 0 0"/>
     </joint>
+    <!-- link: antenna -->
+    <link name="antenna_link">
+        <visual>
+            <geometry>
+                <cylinder length="${antenna_len}" radius="${antenna_rad}"/>
+            </geometry>
+            <origin rpy="0 0 0" xyz="0 0 ${ antenna_len/2}"/>
+        <material name="black"/>
+        </visual>
+        <collision>
+            <geometry>
+                <cylinder length="${antenna_len}" radius="${antenna_rad}"/>
+            </geometry>
+            <origin rpy="0 0 0" xyz="0 0 ${ antenna_len/2}"/>
+        </collision>
+        <xacro:default_inertial mass="0.05"/>
+    </link>
+    <gazebo reference="antenna_link">
+            <material>Gazebo/Yellow </material>
+    </gazebo>
+    <joint name="antenna_joint" type="fixed">
+        <parent link="level_1_link"/>
+        <child link="antenna_link"/>
+        <origin rpy="0 0 0" xyz="${width/2 - antenna_space} ${height/2  - antenna_space} ${level_depth/2}"/>
+    </joint>
+    <!-- gazebo plugin -->
     <gazebo>
         <plugin name="gazebo_ros_control" filename="libgazebo_ros_control.so">

Commit message: add new feature to the gazebo robot
this new feature has been binded to the controller

File: ros/pouco2000_gazebo/urdf/pouco2000.urdf.xacro (robot description, xacro)
@@ -27,4 +27,8 @@
     <xacro:property name="antenna_rad" value="0.01"/>
     <xacro:property name="antenna_space" value="0.1"/>
+    <xacro:property name="disc_len" value="0.02"/>
+    <xacro:property name="disc_rad" value="${width/3}"/>
+    <xacro:property name="disc_depth" value="0.05"/>
+    <xacro:property name="disc_scale" value="0.05"/>
     <!-- colors definitions -->
     <material name="blue">
@@ -277,5 +281,5 @@
         <visual>
             <geometry>
-                <box size="${fork_base_width} ${height} ${depth/10}"/>
+                <box size="${fork_base_width - free_space} ${height - free_space} ${depth/10}"/>
             </geometry>
         <material name="blue"/>
@@ -283,5 +287,5 @@
         <collision>
             <geometry>
-                  <box size="${fork_base_width} ${height} ${depth/10}"/>
+                  <box size="${fork_base_width - free_space} ${height - free_space} ${depth/10}"/>
             </geometry>
         </collision>
@@ -423,4 +427,69 @@
         <origin rpy="0 0 0" xyz="${width/2 - antenna_space} ${height/2  - antenna_space} ${level_depth/2}"/>
     </joint>
+    <!-- links: disk -->
+    <link name="disc_base_link">
+        <visual>
+            <geometry>
+                <box size="${fork_base_width - free_space} ${height - free_space} ${depth/10}"/>
+            </geometry>
+        <material name="blue"/>
+        </visual>
+        <collision>
+            <geometry>
+                  <box size="${fork_base_width - free_space} ${height - free_space} ${depth/10}"/>
+            </geometry>
+        </collision>
+        <xacro:default_inertial mass="1"/>
+    </link>
+    <transmission name="disc_base_trans">
+        <type>transmission_interface/SimpleTransmission</type>
+        <actuator name="disc_base_motor">
+            <mechanicalReduction>1</mechanicalReduction>
+        </actuator>
+        <joint name="disc_base_joint">
+        <hardwareInterface>PositionJointInterface</hardwareInterface>
+        </joint>
+    </transmission>
+    <joint name="disc_base_joint" type="prismatic">
+        <axis rpy="0 0 0" xyz="1 0 0"/>
+        <parent link="base_link"/>
+        <child link="disc_base_link"/>
+        <limit effort="10" lower="0" upper="${disc_rad}" velocity="0.5"/>
+        <origin xyz="${(width)/2 - disc_rad - free_space - fork_base_width/2} 0 ${-1*disc_depth}"/>
+    </joint>
+    <link name="disc_link">
+        <visual>
+            <geometry>
+                <mesh filename="package://pouco2000_gazebo/meshes/disc/disc.STL" scale="${disc_scale} ${disc_scale} ${disc_scale}"/>
+            </geometry>
+            <origin rpy="0 0 0" xyz="-0.3 -0.3 0"/>
+        <material name="blue"/>
+        </visual>
+        <collision>
+            <geometry>
+                <mesh filename="package://pouco2000_gazebo/meshes/disc/disc.STL" scale="${disc_scale} ${disc_scale} ${disc_scale}"/>
+            </geometry>
+        </collision>
+        <xacro:default_inertial mass="1"/>
+    </link>
+    <transmission name="disc_trans">
+        <type>transmission_interface/SimpleTransmission</type>
+        <actuator name="disc_motor">
+            <mechanicalReduction>1</mechanicalReduction>
+        </actuator>
+        <joint name="disc_joint">
+        <hardwareInterface>VelocityJointInterface</hardwareInterface>
+        </joint>
+    </transmission>
+    <joint name="disc_joint" type="continuous">
+        <parent link="disc_base_link"/>
+        <child link="disc_link"/>
+        <axis rpy="0 0 0" xyz="0 0 1"/>
+    </joint>
+    <gazebo reference="disc_link">
+            <material>
+              Gazebo/Grey
+            </material>
+    </gazebo>
     <!-- gazebo plugin -->
     <gazebo>
